File: Loadcell_PCB.kicad_pcb (KiCad board)
At the start: 2 copper layers, 57.5 x 74.6 mm, 53 parts, among them J1 USB_C_Receptacle_USB2.0, J2 Load cell side, J3 Micro_SD_Card, J4 GPS, Q1 S8550, SW1 RESET, U1 ATmega328P-M, U2 CH340C, U3 HX711, U4 74125, U5 LD1117S33TR_SOT223, Y1 16MHz

Commit message: Update unsaved record to the current commit
Changed lines of the file:
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@@
 		(tags "Through hole angled pin header THT 1x02 2.54mm single row")
 		(property "Reference" "J4"
-			(at 4.385 -2.27 -90)
+			(at 2.6416 -2.413 0)
 			(layer "F.SilkS")
 			(effects
